File: Kicad_Projects.kicad_pcb (KiCad board)
At the start: 2 copper layers, 100.3 x 50.8 mm, 30 parts, among them J1 Ent. 15Vca, J2 Vcc_Volt/Amper, J3 Vout, J4 Amperimetro, Q1 BD137, Q2 TIP3055G, U1 LM723_DIP14

Commit message: Actualizacion Jumper 01/06
Parts:
- added JUMPER: Jumper_2_Bridged, Resistor_THT:R_Axial_DIN0207_L6.3mm_D2.5mm_P10.16mm_Horizontal, F.Cu at (145.4, 76.5)
- moved AC_IN 2.54 mm to (84.6, 117.6)
- moved -AMP_METER+ 1.62 mm to (159.8, 105.6)
- moved C6 0.40 mm to (159.8, 87.7)
- renumbered J2 to +DC_METER-, J4 to -AMP_METER+, J3 to -DC_OUT+, J1 to AC_IN, Ajuste_Iout_max1 to Ajuste_Iout_max, Regulacion_Corriente1 to Regulacion_Corriente, Regulacion_Tension1 to Regulacion_Tension
Connections:
- U1 pad 3: Vout -> Net-(U1-Pad3)
Routing:
- net Vout: track 77.4 -> 49.3 mm, vias 2 -> 0
- net Net-(U1-Pad3): track 0.00 -> 17.9 mm
- net AC_F: track 43.8 -> 49.1 mm
- net AC_N: track 41.0 -> 43.3 mm
- net Vout_amp: track 6.86 -> 5.24 mm
Other:
- board text removed: "Jumper"
